Commit message: added an object to the scene and made Mujoco run with head.

File: cartesian_controller_simulation/urdf/robot.urdf.xacro (robot description, xacro)
@@ -68,4 +68,16 @@
                 <origin xyz="0.0 0.0 0.0" rpy="0.0 0.0 0.0" />
         </joint>
+        <joint name="world_joint_cp" type="fixed">
+                <parent link="world" />
+                <child link = "cp_prob_plate" />
+                <origin xyz="1.0 0.5 0.0" rpy="0.0 0.0 0.0" />
+        </joint>
+        <link name="cp_prob_plate" >
+                <visual name="plate">
+                        <geometry>
+                                <box size="0.5 0.05 0.5"/>
+                        </geometry>
+                </visual>
+        </link>
         <link name="base_link" >
                 <inertial>
